Commit message: enable arms

File: resources/robots/h1_2/h1_2_12dof.urdf (robot description, URDF)
Before this commit: robot h1_5, 56 links, 55 joints
Joints:
- joint left_elbow_pitch_joint: type fixed -> revolute
- joint left_elbow_roll_joint: type fixed -> revolute
- joint left_shoulder_pitch_joint: type fixed -> revolute
- joint left_shoulder_roll_joint: type fixed -> revolute
- joint left_shoulder_yaw_joint: type fixed -> revolute
- joint left_wrist_pitch_joint: type fixed -> revolute
- joint left_wrist_yaw_joint: type fixed -> revolute
- joint right_elbow_pitch_joint: type fixed -> revolute
- joint right_elbow_roll_joint: type fixed -> revolute
- joint right_shoulder_pitch_joint: type fixed -> revolute
- joint right_shoulder_roll_joint: type fixed -> revolute
- joint right_shoulder_yaw_joint: type fixed -> revolute
- joint right_wrist_pitch_joint: type fixed -> revolute
- joint right_wrist_yaw_joint: type fixed -> revolute
- joint torso_joint: type fixed -> revolute
